Commit message: add new camera mount to urdf

File: xarm_description/urdf/camera/realsense_d435i.urdf.xacro (robot description, xacro)
@@ -6,10 +6,12 @@
     <link name="${prefix}link_eef">
       <xacro:common_link_visual
-        mesh_filename="camera/realsense/visual/d435_with_cam_stand"
+        mesh_filename="camera/realsense/visual/d435_with_cam_stand_new_with_wire"
+        scale="0.001 0.001 0.001"
         origin_xyz="0 0 0"
         origin_rpy="0 0 0"
         material_name="${prefix}Silver" />
       <xacro:common_link_collision
-        mesh_filename="camera/realsense/collision/d435_with_cam_stand"
+        mesh_filename="camera/realsense/collision/d435_with_cam_stand_new_with_wire"
+        scale="0.001 0.001 0.001"
         origin_xyz="0 0 0"
         origin_rpy="0 0 0" />
@@ -28,5 +30,5 @@
         <parent link="${prefix}link_eef" />
         <child link="${prefix}camera_link" />
-        <origin xyz="0.06746 -0.0175 0.0237" rpy="${M_PI} ${-M_PI/2} 0" />
+        <origin xyz="0.1 -0.0175 0.0267" rpy="${M_PI} ${-M_PI/2} 0" />
       </joint>
       <joint name="${prefix}camera_depth_joint" type="fixed">

File: xarm_description/urdf/common/common.link.xacro (robot description, xacro)
@@ -24,16 +24,16 @@
     </xacro:unless>
   </xacro:macro>
-  <xacro:macro name="common_link_visual" params="mesh_filename add_mesh_suffix:=true material_name:='White' origin_xyz:='0 0 0' origin_rpy:='0 0 0' other_mesh_suffix:=''">
+  <xacro:macro name="common_link_visual" params="mesh_filename add_mesh_suffix:=true material_name:='White' origin_xyz:='0 0 0' origin_rpy:='0 0 0' other_mesh_suffix:='' scale='1.0 1.0 1.0'">
     <visual>
       <geometry>
         <xacro:if value="${add_mesh_suffix}">
-          <mesh filename="${mesh_path}/${mesh_filename}.${mesh_suffix}"/>
+          <mesh filename="${mesh_path}/${mesh_filename}.${mesh_suffix}" scale="${scale}"/>
         </xacro:if>
         <xacro:unless value="${add_mesh_suffix}">
           <xacro:if value="${other_mesh_suffix != ''}">
-            <mesh filename="${mesh_path}/${mesh_filename}.${other_mesh_suffix}"/>
+            <mesh filename="${mesh_path}/${mesh_filename}.${other_mesh_suffix}" scale="${scale}"/>
           </xacro:if>
           <xacro:unless value="${other_mesh_suffix != ''}">
-            <mesh filename="${mesh_path}/${mesh_filename}"/>
+            <mesh filename="${mesh_path}/${mesh_filename}" scale="${scale}"/>
           </xacro:unless>
         </xacro:unless>
@@ -43,16 +43,16 @@
     </visual>
   </xacro:macro>
-  <xacro:macro name="common_link_collision" params="mesh_filename add_mesh_suffix:=true origin_xyz:='0 0 0' origin_rpy:='0 0 0' other_mesh_suffix:=''">
+  <xacro:macro name="common_link_collision" params="mesh_filename add_mesh_suffix:=true origin_xyz:='0 0 0' origin_rpy:='0 0 0' other_mesh_suffix:='' scale='1.0 1.0 1.0'">
     <collision>
       <geometry>
         <xacro:if value="${add_mesh_suffix}">
-          <mesh filename="${mesh_path}/${mesh_filename}.${mesh_suffix}"/>
+          <mesh filename="${mesh_path}/${mesh_filename}.${mesh_suffix}" scale="${scale}"/>
         </xacro:if>
         <xacro:unless value="${add_mesh_suffix}">
           <xacro:if value="${other_mesh_suffix != ''}">
-            <mesh filename="${mesh_path}/${mesh_filename}.${other_mesh_suffix}"/>
+            <mesh filename="${mesh_path}/${mesh_filename}.${other_mesh_suffix}" scale="${scale}"/>
           </xacro:if>
           <xacro:unless value="${other_mesh_suffix != ''}">
-            <mesh filename="${mesh_path}/${mesh_filename}"/>
+            <mesh filename="${mesh_path}/${mesh_filename}" scale="${scale}"/>
           </xacro:unless>
         </xacro:unless>
