Commit message: urdf changes - change base_link to link_base_fixed - realsense urdf to use mesh file without wire to prevent moveit detecting false self collisions with the solid "wire" mesh - constrain joint angle limits further to match the ones on the xarm UI to prevent moveit from planning trajectories that would cause a joint angle error on the xarm

File: xarm_description/urdf/camera/realsense_d435i.urdf (original).xacro (robot description, xacro)
@@ -6,12 +6,10 @@
     <link name="${prefix}link_eef">
       <xacro:common_link_visual
-        mesh_filename="camera/realsense/visual/d435_with_cam_stand_new"
-        scale="0.001 0.001 0.001"
+        mesh_filename="camera/realsense/visual/d435_with_cam_stand"
         origin_xyz="0 0 0"
         origin_rpy="0 0 0"
         material_name="${prefix}Silver" />
       <xacro:common_link_collision
-        mesh_filename="camera/realsense/collision/d435_with_cam_stand_new"
-        scale="0.001 0.001 0.001"
+        mesh_filename="camera/realsense/collision/d435_with_cam_stand"
         origin_xyz="0 0 0"
         origin_rpy="0 0 0" />
@@ -30,5 +28,5 @@
         <parent link="${prefix}link_eef" />
         <child link="${prefix}camera_link" />
-        <origin xyz="0.1 -0.0175 0.0267" rpy="${M_PI} ${-M_PI/2} 0" />
+        <origin xyz="0.06746 -0.0175 0.0237" rpy="${M_PI} ${-M_PI/2} 0" />
       </joint>
       <joint name="${prefix}camera_depth_joint" type="fixed">

File: xarm_description/urdf/xarm6/xarm6_robot_macro.xacro (robot description, xacro)
@@ -34,14 +34,15 @@
           baud_checkset="${baud_checkset}" default_gripper_baud="${default_gripper_baud}"
           joint1_lower_limit="${-pi*0.99}" joint1_upper_limit="${pi*0.99}"
-          joint2_lower_limit="${-2.059}" joint2_upper_limit="${2.0944}"
-          joint3_lower_limit="${-pi*0.99}" joint3_upper_limit="${0.19198}"
+          joint2_lower_limit="${-2.00712}" joint2_upper_limit="${2.00712}"
+          joint3_lower_limit="${-pi*0.99}" joint3_upper_limit="${0.15708}"
           joint4_lower_limit="${-pi*0.99}" joint4_upper_limit="${pi*0.99}"
           joint5_lower_limit="${-1.69297}" joint5_upper_limit="${pi*0.99}"
-          joint6_lower_limit="${-pi*0.99}" joint6_upper_limit="${pi*0.99}"/>
+          joint6_lower_limit="${-pi*0.99}" joint6_upper_limit="${pi*0.99}"
+          />
       </xacro:if>
       <xacro:xarm6_urdf prefix="${prefix}"
         joint1_lower_limit="${-pi*0.99}" joint1_upper_limit="${pi*0.99}"
-        joint2_lower_limit="${-2.059}" joint2_upper_limit="${2.0944}"
-        joint3_lower_limit="${-pi*0.99}" joint3_upper_limit="${0.19198}"
+        joint2_lower_limit="${-2.00712}" joint2_upper_limit="${2.00712}"
+        joint3_lower_limit="${-pi*0.99}" joint3_upper_limit="${0.15708}"
         joint4_lower_limit="${-pi*0.99}" joint4_upper_limit="${pi*0.99}"
         joint5_lower_limit="${-1.69297}" joint5_upper_limit="${pi*0.99}"

File: xarm_description/urdf/xarm_device_macro.xacro (robot description, xacro)
@@ -65,6 +65,6 @@
     <xacro:property name="model_num" value="${scope_parent_model_num}"/>
     <!-- add one world link if no 'attach_to' specified  -->
-    <xacro:if value="${attach_to == 'base_link' and create_attach_link}">
-      <link name="base_link" />
+    <xacro:if value="${attach_to == 'link_base_fixed' and create_attach_link}">
+      <link name="link_base_fixed" />
     </xacro:if>
     <joint name="${prefix}world_joint" type="fixed">
