Commit message: change parent frame of link_base from world to base_link to integrate with mobile base

File: xarm_description/urdf/xarm_device_macro.xacro (robot description, xacro)
@@ -65,6 +65,6 @@
     <xacro:property name="model_num" value="${scope_parent_model_num}"/>
     <!-- add one world link if no 'attach_to' specified  -->
-    <xacro:if value="${attach_to == 'world' and create_attach_link}">
-      <link name="world" />
+    <xacro:if value="${attach_to == 'base_link' and create_attach_link}">
+      <link name="base_link" />
     </xacro:if>
     <joint name="${prefix}world_joint" type="fixed">
