Commit message: add simplified collision geometry to xarm6 urdf

File: xarm_description/urdf/xarm6/xarm6.urdf.xacro (robot description, xacro)
@@ -22,5 +22,5 @@
     <xacro:unless value="${model_num >= 1305 and model_num != 1380}">
       <xacro:property name="visual_dir" value="xarm6/visual"/>
-      <xacro:property name="collision_dir" value="xarm6/visual"/>
+      <xacro:property name="collision_dir" value="xarm6/collision"/>
       <xacro:property name="add_mesh_suffix" value="true"/>
       <xacro:property name="collison_mesh_suffix" value="stl"/>
