Commit message: add ft sensor to urdf

File: xarm_description/urdf/other/other_geometry.urdf.xacro (robot description, xacro)
@@ -40,8 +40,8 @@
         <xacro:property name="_tcp_z" value="${geometry_radius * 2}"/>
       </xacro:unless>
-      <xacro:property name="_origin_xyz" value="0 0 ${_origin_y}"/>
-      <xacro:property name="_origin_rpy" value="0 0 0"/>
-      <xacro:property name="_tcp_xyz" value="0 0 ${_tcp_z}"/>
-      <xacro:property name="_tcp_rpy" value="0 0 0"/>
+      <xacro:property name="_origin_xyz" value="${geometry_mesh_origin_xyz}"/>
+      <xacro:property name="_origin_rpy" value="${geometry_mesh_origin_rpy}"/>
+      <xacro:property name="_tcp_xyz" value="${geometry_mesh_tcp_xyz}"/>
+      <xacro:property name="_tcp_rpy" value="${geometry_mesh_tcp_rpy}"/>
     </xacro:unless>
     <xacro:if value="${geometry_mesh_filename.startswith('file:///') or geometry_mesh_filename.startswith('package://')}">

File: xarm_description/urdf/xarm_device_macro.xacro (robot description, xacro)
@@ -214,5 +214,5 @@
     </xacro:unless>
     <joint name="${prefix}joint_eef" type="fixed">
-      <origin xyz="0 0 0" rpy="0 0 0" />
+      <origin xyz="0 0 0.06" rpy="0 0 0" />
       <parent link="${prefix}link${dof}" />
       <child link="${prefix}link_eef" />
@@ -263,4 +263,7 @@
       />
     </xacro:if>
+    <!-- Load FT sensor URDF -->
+    <xacro:include filename="$(find xarm_description)/urdf/other/ft_sensor.urdf.xacro" />
+    <xacro:ft_sensor prefix="${prefix}" attach_to="${prefix}link6"/>
     <!-- gazebo_plugin -->
     <xacro:if value="${load_gazebo_plugin}">

File: xarm_moveit_config/srdf/_xarm6_macro.srdf.xacro (robot description, xacro)
@@ -82,4 +82,5 @@
       <passive_joint name="${prefix}right_outer_knuckle_joint" />
       <passive_joint name="${prefix}right_finger_joint" />
+      <passive_joint name="${prefix}ft_sensor_joint" />
       <!-- DISABLE COLLISIONS, By default it is assumed that any link of the robot could potentially come into collision with any other link in the robot. This tag disables collision checking between a specified pair of links. -->
       <disable_collisions link1="${prefix}left_finger" link2="${prefix}left_inner_knuckle" reason="Default" />
@@ -202,4 +203,5 @@
     <disable_collisions link1="${prefix}link5" link2="${prefix}link6" reason="Adjacent" />
     <disable_collisions link1="${prefix}link6" link2="${prefix}link_eef" reason="Adjacent" />
+    <disable_collisions link1="${prefix}link6" link2="${prefix}ft_sensor_link" reason="Adjacent" />
   </xacro:macro>
 </robot>
